File: processing/and_or_matrix/circuit/circuit.sch (EAGLE design)
At the start: 61 parts, among them IC1 74HC04, IC2 74HC04, IC3 74HC21N, IC4 74HC21N, IC5 74HC32

Commit message: updated processing unit   + minor changes (renamed some resistors, added some values, moved names of leds)   + added parts
Parts:
- RPU1, RPU2, RPU3, RPU4: value (none) -> 10k
- renumbered RN6 to RPU2, RN7 to RPU1, RN8 to RPU3, RN9 to RPU4
